File: hardware/kicad/shipometer.kicad_pcb (KiCad board)
At the start: 2 copper layers, 65 x 71.6 mm, 66 parts, among them J101 Raspberry_Pi_40, J102 Conn_01x03, J104 ICM20948, J105 BME280, J106 ZED-F9R, J701 Conn_01x06_Pin, J702 Conn_01x06_Pin, J703 Conn_01x06_Pin, J704 Conn_01x06_Pin, U102 74LS138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

Commit message: Change version number to 23.04.1 reflecting the green-wire fix
Other:
- board text added: "Version 23.04.1"
- board text removed: "Version 23.05"
Changed lines of the file:
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@@
 		)
 	)
-	(gr_text "Version 23.05"
+	(gr_text "Version 23.04.1"
 		(at 154.178 84.836 0)
 		(layer "F.Mask")
@@
 		)
 	)
-	(gr_text "Version 23.05"
+	(gr_text "Version 23.04.1"
 		(at 164.592 84.836 0)
 		(layer "B.Mask")
